File: auv_1.kicad_sch (KiCad schematic)
At the start: 21 parts, among them U1 RASPBERRY_PI_PICO_W

Commit message: Schematic Updated
Connections:
- net at 12V_3.3V. (Vout_n): now also 16V_12V. (Vout_n), Jetson1. (Gnd)
- new net: 12V_3.3V. (Vout_n), Jetson1. (Gnd), Small_Relay. (NC), T1. (NO), T2. (NO), T3. (NO), T4. (NO), T5. (NO), T6. (NO)
- new net: ESC6. (-ve), T6. (NO)
- new net: 16V_12V. (Vout_n), Small_Relay. (NC), T1. (NO), T2. (NO), T3. (NO), T4. (NO), T5. (NO), T6. (NO)
- new net: ESC5. (-ve), T5. (NO)
- new net: ESC4. (-ve), T4. (NO)
- new net: ESC3. (-ve), T3. (NO)
- new net: 16V_5V. (Vout_n), Kill_switch. (DO), Small_Relay. (NC) (x2)
- new net: ESC2. (-ve), T2. (NO)
- new net: ESC1. (-ve), T1. (NO)
- now unconnected: Small_Relay. (NC), Small_Relay. (NC), Small_Relay. (NC), Small_Relay. (NC)
Changed lines of the file:
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@@
+	(wire
+		(pts
+			(xy 237.49 288.29) (xy 234.95 288.29)
+		)
+		(stroke
+			(width 0)
+			(type default)
+		)
+	)
 	(wire
 		(pts
@@
 	(wire
 		(pts
+			(xy 281.94 300.99) (xy 281.94 287.02)
+		)
+		(stroke
+			(width 0)
+			(type default)
+		)
+	)
+	(wire
+		(pts
+			(xy 135.89 289.56) (xy 144.78 289.56)
+		)
+		(stroke
+			(width 0)
+			(type default)
+		)
+	)
+	(wire
+		(pts
 			(xy 279.4 274.32) (xy 280.67 274.32)
 		)
@@
 	(wire
 		(pts
-			(xy 326.39 281.94) (xy 326.39 302.26)
-		)
-		(stroke
-			(width 0)
-			(type default)
-		)
-	)
-	(wire
-		(pts
 			(xy 205.74 318.77) (xy 205.74 312.42)
 		)
@@
 	(wire
 		(pts
+			(xy 194.31 318.77) (xy 194.31 289.56)
+		)
+		(stroke
+			(width 0)
+			(type default)
+		)
+	)
+	(wire
+		(pts
 			(xy 200.66 224.79) (xy 276.86 224.79)
 		)
@@
 	(wire
 		(pts
+			(xy 281.94 287.02) (xy 279.4 287.02)
+		)
+		(stroke
+			(width 0)
+			(type default)
+		)
+	)
+	(wire
+		(pts
 			(xy 135.89 276.86) (xy 138.43 276.86)
 		)
@@
 	(wire
 		(pts
-			(xy 144.78 283.21) (xy 144.78 314.96)
+			(xy 194.31 289.56) (xy 189.23 289.56)
+		)
+		(stroke
+			(width 0)
+			(type default)
+		)
+	)
+	(wire
+		(pts
+			(xy 144.78 289.56) (xy 144.78 314.96)
 		)
 		(stroke
@@
 	(wire
 		(pts
+			(xy 326.39 302.26) (xy 326.39 288.29)
+		)
+		(stroke
+			(width 0)
+			(type default)
+		)
+	)
+	(wire
+		(pts
 			(xy 323.85 176.53) (xy 323.85 182.88)
 		)
@@
 	(wire
 		(pts
-			(xy 322.58 281.94) (xy 326.39 281.94)
-		)
-		(stroke
-			(width 0)
-			(type default)
-		)
-	)
-	(wire
-		(pts
 			(xy 280.67 92.71) (xy 346.71 92.71)
 		)
@@
 	(wire
 		(pts
+			(xy 369.57 287.02) (xy 367.03 287.02)
+		)
+		(stroke
+			(width 0)
+			(type default)
+		)
+	)
+	(wire
+		(pts
 			(xy 373.38 250.19) (xy 373.38 321.31)
 		)
@@
 	(wire
 		(pts
-			(xy 234.95 281.94) (xy 237.49 281.94)
-		)
-		(stroke
-			(width 0)
-			(type default)
-		)
-	)
-	(wire
-		(pts
 			(xy 273.05 179.07) (xy 377.19 179.07)
 		)
@@
 	(wire
 		(pts
-			(xy 194.31 283.21) (xy 194.31 318.77)
-		)
-		(stroke
-			(width 0)
-			(type default)
-		)
-	)
-	(wire
-		(pts
-			(xy 281.94 280.67) (xy 281.94 300.99)
-		)
-		(stroke
-			(width 0)
-			(type default)
-		)
-	)
-	(wire
-		(pts
 			(xy 104.14 259.08) (xy 157.48 259.08)
 		)
@@
 	(wire
 		(pts
+			(xy 326.39 288.29) (xy 322.58 288.29)
+		)
+		(stroke
+			(width 0)
+			(type default)
+		)
+	)
+	(wire
+		(pts
 			(xy 243.84 226.06) (xy 243.84 320.04)
 		)
@@
 	(wire
 		(pts
-			(xy 189.23 283.21) (xy 194.31 283.21)
-		)
-		(stroke
-			(width 0)
-			(type default)
-		)
-	)
-	(wire
-		(pts
 			(xy 281.94 176.53) (xy 281.94 228.6)
 		)
@@
 	(wire
 		(pts
+			(xy 237.49 300.99) (xy 237.49 288.29)
+		)
+		(stroke
+			(width 0)
+			(type default)
+		)
+	)
+	(wire
+		(pts
 			(xy 280.67 274.32) (xy 280.67 270.51)
 		)
@@
 	(wire
 		(pts
-			(xy 367.03 280.67) (xy 369.57 280.67)
-		)
-		(stroke
-			(width 0)
-			(type default)
-		)
-	)
-	(wire
-		(pts
 			(xy 234.95 300.99) (xy 234.95 320.04)
 		)
@@
 	(wire
 		(pts
+			(xy 369.57 321.31) (xy 369.57 287.02)
+		)
+		(stroke
+			(width 0)
+			(type default)
+		)
+	)
+	(wire
+		(pts
 			(xy 290.83 306.07) (xy 335.28 306.07)
 		)
@@
 	(wire
 		(pts
-			(xy 135.89 283.21) (xy 144.78 283.21)
-		)
-		(stroke
-			(width 0)
-			(type default)
-		)
-	)
-	(wire
-		(pts
 			(xy 280.67 105.41) (xy 297.18 105.41)
 		)
@@
 	(wire
 		(pts
-			(xy 369.57 280.67) (xy 369.57 321.31)
-		)
-		(stroke
-			(width 0)
-			(type default)
-		)
-	)
-	(wire
-		(pts
-			(xy 237.49 281.94) (xy 237.49 300.99)
-		)
-		(stroke
-			(width 0)
-			(type default)
-		)
-	)
-	(wire
-		(pts
 			(xy 166.37 158.75) (xy 176.53 158.75)
 		)
@@
 		)
 		(stroke
-			(width 0)
-			(type default)
-		)
-	)
-	(wire
-		(pts
-			(xy 279.4 280.67) (xy 281.94 280.67)
-		)
-		(stroke
